File: MCP2518.sch (KiCad schematic (older format))
At the start: 10 parts, among them U1 MCP2518FDT-H_SL, U2 SN65HVD231, Y1 XRCGB40M000F4M02R0

Commit message: EN Pullup, DTR + RTS
Parts:
- C4, C5: footprint Resistor_SMD:R_0603_1608Metric -> Capacitor_SMD:C_0603_1608Metric
Changed lines of the file:
@@
 F 0 "C4" H 6292 1696 50  0000 L CNN
 F 1 "0.1uF" H 6292 1605 50  0000 L CNN
-F 2 "Resistor_SMD:R_0603_1608Metric" H 6200 1650 50  0001 C CNN
+F 2 "Capacitor_SMD:C_0603_1608Metric" H 6200 1650 50  0001 C CNN
 F 3 "~" H 6200 1650 50  0001 C CNN
 	1    6200 1650
@@
 F 0 "C5" H 7892 3046 50  0000 L CNN
 F 1 "0.1uF" H 7892 2955 50  0000 L CNN
-F 2 "Resistor_SMD:R_0603_1608Metric" H 7800 3000 50  0001 C CNN
+F 2 "Capacitor_SMD:C_0603_1608Metric" H 7800 3000 50  0001 C CNN
 F 3 "~" H 7800 3000 50  0001 C CNN
 	1    7800 3000

Commit message: ESP32 Bus extrahiert
Parts:
- R6: footprint Resistor_SMD:R_1206_3216Metric_Pad1.30x1.75mm_HandSolder -> Resistor_SMD:R_0603_1608Metric
Changed lines of the file:
@@
 F 0 "R6" H 7609 2446 50  0000 L CNN
 F 1 "120" H 7609 2355 50  0000 L CNN
-F 2 "Resistor_SMD:R_1206_3216Metric_Pad1.30x1.75mm_HandSolder" H 7550 2400 50  0001 C CNN
+F 2 "Resistor_SMD:R_0603_1608Metric" H 7550 2400 50  0001 C CNN
 F 3 "~" H 7550 2400 50  0001 C CNN
 	1    7550 2400
